File: calico_cpu/ctl_logic.kicad_sch (KiCad schematic)
At the start: 6 parts, among them U46 74HC02, U47 74HC21, U48 74HC00

Commit message: calico_cpu: assign footprints
Parts:
- C46, C47, C48: footprint (none) -> Capacitor_SMD:C_0805_2012Metric_Pad1.18x1.45mm_HandSolder
- U46, U47, U48: footprint (none) -> PrjLibrary:DIP-14_W7.62mm_D1mm
Changed lines of the file:
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@@
     (property "Reference" "U46" (id 0) (at 41.91 78.74 0))
     (property "Value" "74HC02" (id 1) (at 41.91 81.28 0))
-    (property "Footprint" "" (id 2) (at 41.91 87.63 0)
+    (property "Footprint" "PrjLibrary:DIP-14_W7.62mm_D1mm" (id 2) (at 41.91 87.63 0)
       (effects (font (size 1.27 1.27)) hide)
     )
@@
     (property "Reference" "U46" (id 0) (at 41.91 60.96 0))
     (property "Value" "74HC02" (id 1) (at 41.91 63.5 0))
-    (property "Footprint" "" (id 2) (at 41.91 69.85 0)
+    (property "Footprint" "PrjLibrary:DIP-14_W7.62mm_D1mm" (id 2) (at 41.91 69.85 0)
       (effects (font (size 1.27 1.27)) hide)
     )
@@
       (effects (font (size 1.27 1.27)) (justify left))
     )
-    (property "Footprint" "" (id 2) (at 74.93 165.1 0)
+    (property "Footprint" "PrjLibrary:DIP-14_W7.62mm_D1mm" (id 2) (at 74.93 165.1 0)
       (effects (font (size 1.27 1.27)) hide)
     )
@@
       (effects (font (size 1.27 1.27)) (justify left))
     )
-    (property "Footprint" "" (id 2) (at 202.8952 151.13 0)
+    (property "Footprint" "Capacitor_SMD:C_0805_2012Metric_Pad1.18x1.45mm_HandSolder" (id 2) (at 202.8952 151.13 0)
       (effects (font (size 1.27 1.27)) hide)
     )
@@
     (property "Reference" "U48" (id 0) (at 156.21 107.95 0))
     (property "Value" "74HC00" (id 1) (at 156.21 110.49 0))
-    (property "Footprint" "" (id 2) (at 156.21 116.84 0)
+    (property "Footprint" "PrjLibrary:DIP-14_W7.62mm_D1mm" (id 2) (at 156.21 116.84 0)
       (effects (font (size 1.27 1.27)) hide)
     )
@@
       (effects (font (size 1.27 1.27)) (justify left))
     )
-    (property "Footprint" "" (id 2) (at 214.3252 151.13 0)
+    (property "Footprint" "Capacitor_SMD:C_0805_2012Metric_Pad1.18x1.45mm_HandSolder" (id 2) (at 214.3252 151.13 0)
       (effects (font (size 1.27 1.27)) hide)
     )
@@
     (property "Reference" "U47" (id 0) (at 80.01 63.5 0))
     (property "Value" "74HC21" (id 1) (at 80.01 66.04 0))
-    (property "Footprint" "" (id 2) (at 80.01 73.66 0)
+    (property "Footprint" "PrjLibrary:DIP-14_W7.62mm_D1mm" (id 2) (at 80.01 73.66 0)
       (effects (font (size 1.27 1.27)) hide)
     )
@@
     (property "Reference" "U46" (id 0) (at 41.91 114.3 0))
     (property "Value" "74HC02" (id 1) (at 41.91 116.84 0))
-    (property "Footprint" "" (id 2) (at 41.91 123.19 0)
+    (property "Footprint" "PrjLibrary:DIP-14_W7.62mm_D1mm" (id 2) (at 41.91 123.19 0)
       (effects (font (size 1.27 1.27)) hide)
     )
@@
     (property "Reference" "U48" (id 0) (at 191.77 64.77 0))
     (property "Value" "74HC00" (id 1) (at 191.77 67.31 0))
-    (property "Footprint" "" (id 2) (at 191.77 73.66 0)
+    (property "Footprint" "PrjLibrary:DIP-14_W7.62mm_D1mm" (id 2) (at 191.77 73.66 0)
       (effects (font (size 1.27 1.27)) hide)
     )
@@
     (property "Reference" "U47" (id 0) (at 160.02 66.04 0))
     (property "Value" "74HC21" (id 1) (at 160.02 68.58 0))
-    (property "Footprint" "" (id 2) (at 160.02 76.2 0)
+    (property "Footprint" "PrjLibrary:DIP-14_W7.62mm_D1mm" (id 2) (at 160.02 76.2 0)
       (effects (font (size 1.27 1.27)) hide)
     )
@@
     (property "Reference" "U46" (id 0) (at 41.91 96.52 0))
     (property "Value" "74HC02" (id 1) (at 41.91 99.06 0))
-    (property "Footprint" "" (id 2) (at 41.91 105.41 0)
+    (property "Footprint" "PrjLibrary:DIP-14_W7.62mm_D1mm" (id 2) (at 41.91 105.41 0)
       (effects (font (size 1.27 1.27)) hide)
     )
@@
       (effects (font (size 1.27 1.27)) (justify left))
     )
-    (property "Footprint" "" (id 2) (at 191.4652 151.13 0)
+    (property "Footprint" "Capacitor_SMD:C_0805_2012Metric_Pad1.18x1.45mm_HandSolder" (id 2) (at 191.4652 151.13 0)
       (effects (font (size 1.27 1.27)) hide)
     )
@@
     (property "Reference" "U48" (id 0) (at 111.76 67.31 0))
     (property "Value" "74HC00" (id 1) (at 111.76 69.85 0))
-    (property "Footprint" "" (id 2) (at 111.76 76.2 0)
+    (property "Footprint" "PrjLibrary:DIP-14_W7.62mm_D1mm" (id 2) (at 111.76 76.2 0)
       (effects (font (size 1.27 1.27)) hide)
     )
@@
       (effects (font (size 1.27 1.27)) (justify left))
     )
-    (property "Footprint" "" (id 2) (at 40.64 165.1 0)
+    (property "Footprint" "PrjLibrary:DIP-14_W7.62mm_D1mm" (id 2) (at 40.64 165.1 0)
       (effects (font (size 1.27 1.27)) hide)
     )
@@
     (property "Reference" "U48" (id 0) (at 111.76 85.09 0))
     (property "Value" "74HC00" (id 1) (at 111.76 87.63 0))
-    (property "Footprint" "" (id 2) (at 111.76 93.98 0)
+    (property "Footprint" "PrjLibrary:DIP-14_W7.62mm_D1mm" (id 2) (at 111.76 93.98 0)
       (effects (font (size 1.27 1.27)) hide)
     )
@@
       (effects (font (size 1.27 1.27)) (justify left))
     )
-    (property "Footprint" "" (id 2) (at 113.03 165.1 0)
-      (effects (font (size 1.27 1.27)) hide)
-    )
+    (property "Footprint" "PrjLibrary:DIP-14_W7.62mm_D1mm" (id 2) (at 113.03 165.1 0)
+      (effects (font (size 1.27 1.27)) hide)
+    )
