File: calico_cpu/inst_fetch.kicad_sch (KiCad schematic)
At the start: 6 parts, among them J1 Conn_01x06, J2 Conn_02x10_Top_Bottom, U1 74HC161, U2 74HC161

Commit message: calico_cpu: assign footprints
Parts:
- C1, C2: footprint (none) -> Capacitor_SMD:C_0805_2012Metric_Pad1.18x1.45mm_HandSolder
- J1: footprint (none) -> Connector_PinHeader_2.54mm:PinHeader_1x06_P2.54mm_Vertical
- J2: footprint (none) -> PrjLibrary:PinHeader_2x10_P2.54mm_Vertical_Top_Bottom
- U1, U2: footprint (none) -> PrjLibrary:DIP-16_W7.62mm_D1mm
Changed lines of the file:
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@@
       (effects (font (size 1.27 1.27)) (justify left))
     )
-    (property "Footprint" "" (id 2) (at 226.06 77.47 0)
+    (property "Footprint" "Connector_PinHeader_2.54mm:PinHeader_1x06_P2.54mm_Vertical" (id 2) (at 226.06 77.47 0)
       (effects (font (size 1.27 1.27)) hide)
     )
@@
       (effects (font (size 1.27 1.27)) (justify left))
     )
-    (property "Footprint" "" (id 2) (at 76.2 53.34 0)
+    (property "Footprint" "PrjLibrary:DIP-16_W7.62mm_D1mm" (id 2) (at 76.2 53.34 0)
       (effects (font (size 1.27 1.27)) hide)
     )
@@
       (effects (font (size 1.27 1.27)) (justify left))
     )
-    (property "Footprint" "" (id 2) (at 124.46 53.34 0)
+    (property "Footprint" "PrjLibrary:DIP-16_W7.62mm_D1mm" (id 2) (at 124.46 53.34 0)
       (effects (font (size 1.27 1.27)) hide)
     )
@@
     (property "Reference" "J2" (id 0) (at 227.33 30.48 0))
     (property "Value" "Conn_02x10_Top_Bottom" (id 1) (at 227.33 33.02 0))
-    (property "Footprint" "" (id 2) (at 226.06 46.99 0)
+    (property "Footprint" "PrjLibrary:PinHeader_2x10_P2.54mm_Vertical_Top_Bottom" (id 2) (at 226.06 46.99 0)
       (effects (font (size 1.27 1.27)) hide)
     )
@@
       (effects (font (size 1.27 1.27)) (justify left))
     )
-    (property "Footprint" "" (id 2) (at 239.7252 154.94 0)
+    (property "Footprint" "Capacitor_SMD:C_0805_2012Metric_Pad1.18x1.45mm_HandSolder" (id 2) (at 239.7252 154.94 0)
       (effects (font (size 1.27 1.27)) hide)
     )
@@
       (effects (font (size 1.27 1.27)) (justify left))
     )
-    (property "Footprint" "" (id 2) (at 228.2952 154.94 0)
-      (effects (font (size 1.27 1.27)) hide)
-    )
+    (property "Footprint" "Capacitor_SMD:C_0805_2012Metric_Pad1.18x1.45mm_HandSolder" (id 2) (at 228.2952 154.94 0)
+      (effects (font (size 1.27 1.27)) hide)
+    )
