File: calico_cpu/logic_rr00ss1x.kicad_sch (KiCad schematic)
At the start: 16 parts, among them U24 74HC00, U25 74HC00, U26 74HC153, U27 74HC153, U28 74HC153, U29 74HC153, U30 74HC157, U31 74HC157

Commit message: calico_cpu: assign footprints
Parts:
- C24, C25, C26, C27, C28, C29, C30, C31: footprint (none) -> Capacitor_SMD:C_0805_2012Metric_Pad1.18x1.45mm_HandSolder
- U24, U25: footprint (none) -> PrjLibrary:DIP-14_W7.62mm_D1mm
- U26, U27, U28, U29, U30, U31: footprint (none) -> PrjLibrary:DIP-16_W7.62mm_D1mm
Changed lines of the file:
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@@
       (effects (font (size 1.27 1.27)) (justify left))
     )
-    (property "Footprint" "" (id 2) (at 124.1552 111.76 0)
+    (property "Footprint" "Capacitor_SMD:C_0805_2012Metric_Pad1.18x1.45mm_HandSolder" (id 2) (at 124.1552 111.76 0)
       (effects (font (size 1.27 1.27)) hide)
     )
@@
       (effects (font (size 1.27 1.27)) (justify left))
     )
-    (property "Footprint" "" (id 2) (at 135.5852 111.76 0)
+    (property "Footprint" "Capacitor_SMD:C_0805_2012Metric_Pad1.18x1.45mm_HandSolder" (id 2) (at 135.5852 111.76 0)
       (effects (font (size 1.27 1.27)) hide)
     )
@@
       (effects (font (size 1.27 1.27)) (justify left))
     )
-    (property "Footprint" "" (id 2) (at 237.49 124.46 0)
+    (property "Footprint" "PrjLibrary:DIP-16_W7.62mm_D1mm" (id 2) (at 237.49 124.46 0)
       (effects (font (size 1.27 1.27)) hide)
     )
@@
     (property "Reference" "U24" (id 0) (at 38.1 123.19 0))
     (property "Value" "74HC00" (id 1) (at 38.1 125.73 0))
-    (property "Footprint" "" (id 2) (at 38.1 132.08 0)
+    (property "Footprint" "PrjLibrary:DIP-14_W7.62mm_D1mm" (id 2) (at 38.1 132.08 0)
       (effects (font (size 1.27 1.27)) hide)
     )
@@
       (effects (font (size 1.27 1.27)) (justify left))
     )
-    (property "Footprint" "" (id 2) (at 38.1 175.26 0)
+    (property "Footprint" "PrjLibrary:DIP-14_W7.62mm_D1mm" (id 2) (at 38.1 175.26 0)
       (effects (font (size 1.27 1.27)) hide)
     )
@@
     (property "Reference" "U25" (id 0) (at 73.66 123.19 0))
     (property "Value" "74HC00" (id 1) (at 73.66 125.73 0))
-    (property "Footprint" "" (id 2) (at 73.66 132.08 0)
+    (property "Footprint" "PrjLibrary:DIP-14_W7.62mm_D1mm" (id 2) (at 73.66 132.08 0)
       (effects (font (size 1.27 1.27)) hide)
     )
@@
     (property "Reference" "U24" (id 0) (at 38.1 107.95 0))
     (property "Value" "74HC00" (id 1) (at 38.1 110.49 0))
-    (property "Footprint" "" (id 2) (at 38.1 116.84 0)
+    (property "Footprint" "PrjLibrary:DIP-14_W7.62mm_D1mm" (id 2) (at 38.1 116.84 0)
       (effects (font (size 1.27 1.27)) hide)
     )
@@
       (effects (font (size 1.27 1.27)) (justify left))
     )
-    (property "Footprint" "" (id 2) (at 135.5852 124.46 0)
+    (property "Footprint" "Capacitor_SMD:C_0805_2012Metric_Pad1.18x1.45mm_HandSolder" (id 2) (at 135.5852 124.46 0)
       (effects (font (size 1.27 1.27)) hide)
     )
@@
       (effects (font (size 1.27 1.27)) (justify left))
     )
-    (property "Footprint" "" (id 2) (at 64.77 50.8 0)
+    (property "Footprint" "PrjLibrary:DIP-16_W7.62mm_D1mm" (id 2) (at 64.77 50.8 0)
       (effects (font (size 1.27 1.27)) hide)
     )
@@
     (property "Reference" "U24" (id 0) (at 38.1 138.43 0))
     (property "Value" "74HC00" (id 1) (at 38.1 140.97 0))
-    (property "Footprint" "" (id 2) (at 38.1 147.32 0)
+    (property "Footprint" "PrjLibrary:DIP-14_W7.62mm_D1mm" (id 2) (at 38.1 147.32 0)
       (effects (font (size 1.27 1.27)) hide)
     )
@@
     (property "Reference" "U25" (id 0) (at 73.66 138.43 0))
     (property "Value" "74HC00" (id 1) (at 73.66 140.97 0))
-    (property "Footprint" "" (id 2) (at 73.66 147.32 0)
+    (property "Footprint" "PrjLibrary:DIP-14_W7.62mm_D1mm" (id 2) (at 73.66 147.32 0)
       (effects (font (size 1.27 1.27)) hide)
     )
@@
       (effects (font (size 1.27 1.27)) (justify left))
     )
-    (property "Footprint" "" (id 2) (at 181.61 50.8 0)
+    (property "Footprint" "PrjLibrary:DIP-16_W7.62mm_D1mm" (id 2) (at 181.61 50.8 0)
       (effects (font (size 1.27 1.27)) hide)
     )
@@
       (effects (font (size 1.27 1.27)) (justify left))
     )
-    (property "Footprint" "" (id 2) (at 73.66 175.26 0)
+    (property "Footprint" "PrjLibrary:DIP-14_W7.62mm_D1mm" (id 2) (at 73.66 175.26 0)
       (effects (font (size 1.27 1.27)) hide)
     )
@@
     (property "Reference" "U24" (id 0) (at 38.1 92.71 0))
     (property "Value" "74HC00" (id 1) (at 38.1 95.25 0))
-    (property "Footprint" "" (id 2) (at 38.1 101.6 0)
+    (property "Footprint" "PrjLibrary:DIP-14_W7.62mm_D1mm" (id 2) (at 38.1 101.6 0)
       (effects (font (size 1.27 1.27)) hide)
     )
@@
     (property "Reference" "U25" (id 0) (at 73.66 107.95 0))
     (property "Value" "74HC00" (id 1) (at 73.66 110.49 0))
-    (property "Footprint" "" (id 2) (at 73.66 116.84 0)
+    (property "Footprint" "PrjLibrary:DIP-14_W7.62mm_D1mm" (id 2) (at 73.66 116.84 0)
       (effects (font (size 1.27 1.27)) hide)
     )
@@
       (effects (font (size 1.27 1.27)) (justify left))
     )
-    (property "Footprint" "" (id 2) (at 112.7252 111.76 0)
+    (property "Footprint" "Capacitor_SMD:C_0805_2012Metric_Pad1.18x1.45mm_HandSolder" (id 2) (at 112.7252 111.76 0)
       (effects (font (size 1.27 1.27)) hide)
     )
@@
       (effects (font (size 1.27 1.27)) (justify left))
     )
-    (property "Footprint" "" (id 2) (at 101.2952 124.46 0)
+    (property "Footprint" "Capacitor_SMD:C_0805_2012Metric_Pad1.18x1.45mm_HandSolder" (id 2) (at 101.2952 124.46 0)
       (effects (font (size 1.27 1.27)) hide)
     )
@@
       (effects (font (size 1.27 1.27)) (justify left))
     )
-    (property "Footprint" "" (id 2) (at 120.65 50.8 0)
+    (property "Footprint" "PrjLibrary:DIP-16_W7.62mm_D1mm" (id 2) (at 120.65 50.8 0)
       (effects (font (size 1.27 1.27)) hide)
     )
@@
     (property "Reference" "U25" (id 0) (at 73.66 92.71 0))
     (property "Value" "74HC00" (id 1) (at 73.66 95.25 0))
-    (property "Footprint" "" (id 2) (at 73.66 101.6 0)
+    (property "Footprint" "PrjLibrary:DIP-14_W7.62mm_D1mm" (id 2) (at 73.66 101.6 0)
       (effects (font (size 1.27 1.27)) hide)
     )
@@
       (effects (font (size 1.27 1.27)) (justify left))
     )
-    (property "Footprint" "" (id 2) (at 181.61 124.46 0)
+    (property "Footprint" "PrjLibrary:DIP-16_W7.62mm_D1mm" (id 2) (at 181.61 124.46 0)
       (effects (font (size 1.27 1.27)) hide)
     )
@@
       (effects (font (size 1.27 1.27)) (justify left))
     )
-    (property "Footprint" "" (id 2) (at 237.49 50.8 0)
+    (property "Footprint" "PrjLibrary:DIP-16_W7.62mm_D1mm" (id 2) (at 237.49 50.8 0)
       (effects (font (size 1.27 1.27)) hide)
     )
@@
       (effects (font (size 1.27 1.27)) (justify left))
     )
-    (property "Footprint" "" (id 2) (at 101.2952 111.76 0)
+    (property "Footprint" "Capacitor_SMD:C_0805_2012Metric_Pad1.18x1.45mm_HandSolder" (id 2) (at 101.2952 111.76 0)
       (effects (font (size 1.27 1.27)) hide)
     )
@@
       (effects (font (size 1.27 1.27)) (justify left))
     )
-    (property "Footprint" "" (id 2) (at 112.7252 124.46 0)
+    (property "Footprint" "Capacitor_SMD:C_0805_2012Metric_Pad1.18x1.45mm_HandSolder" (id 2) (at 112.7252 124.46 0)
       (effects (font (size 1.27 1.27)) hide)
     )
@@
       (effects (font (size 1.27 1.27)) (justify left))
     )
-    (property "Footprint" "" (id 2) (at 124.1552 124.46 0)
-      (effects (font (size 1.27 1.27)) hide)
-    )
+    (property "Footprint" "Capacitor_SMD:C_0805_2012Metric_Pad1.18x1.45mm_HandSolder" (id 2) (at 124.1552 124.46 0)
+      (effects (font (size 1.27 1.27)) hide)
+    )
