File: calico_cpu/logic_rr01ss0x.kicad_sch (KiCad schematic)
At the start: 8 parts, among them U32 74HC283, U33 74HC283, U34 74HC157, U35 74HC157

Commit message: calico_cpu: assign footprints
Parts:
- C32, C33, C34, C35: footprint (none) -> Capacitor_SMD:C_0805_2012Metric_Pad1.18x1.45mm_HandSolder
- U32, U33, U34, U35: footprint (none) -> PrjLibrary:DIP-16_W7.62mm_D1mm
Changed lines of the file:
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@@
       (effects (font (size 1.27 1.27)) (justify left))
     )
-    (property "Footprint" "" (id 2) (at 124.46 86.36 0)
+    (property "Footprint" "PrjLibrary:DIP-16_W7.62mm_D1mm" (id 2) (at 124.46 86.36 0)
       (effects (font (size 1.27 1.27)) hide)
     )
@@
       (effects (font (size 1.27 1.27)) (justify left))
     )
-    (property "Footprint" "" (id 2) (at 184.15 88.9 0)
+    (property "Footprint" "PrjLibrary:DIP-16_W7.62mm_D1mm" (id 2) (at 184.15 88.9 0)
       (effects (font (size 1.27 1.27)) hide)
     )
@@
       (effects (font (size 1.27 1.27)) (justify left))
     )
-    (property "Footprint" "" (id 2) (at 214.3252 148.59 0)
+    (property "Footprint" "Capacitor_SMD:C_0805_2012Metric_Pad1.18x1.45mm_HandSolder" (id 2) (at 214.3252 148.59 0)
       (effects (font (size 1.27 1.27)) hide)
     )
@@
       (effects (font (size 1.27 1.27)) (justify left))
     )
-    (property "Footprint" "" (id 2) (at 225.7552 148.59 0)
+    (property "Footprint" "Capacitor_SMD:C_0805_2012Metric_Pad1.18x1.45mm_HandSolder" (id 2) (at 225.7552 148.59 0)
       (effects (font (size 1.27 1.27)) hide)
     )
@@
       (effects (font (size 1.27 1.27)) (justify left))
     )
-    (property "Footprint" "" (id 2) (at 202.8952 148.59 0)
+    (property "Footprint" "Capacitor_SMD:C_0805_2012Metric_Pad1.18x1.45mm_HandSolder" (id 2) (at 202.8952 148.59 0)
       (effects (font (size 1.27 1.27)) hide)
     )
@@
       (effects (font (size 1.27 1.27)) (justify left))
     )
-    (property "Footprint" "" (id 2) (at 68.58 86.36 0)
+    (property "Footprint" "PrjLibrary:DIP-16_W7.62mm_D1mm" (id 2) (at 68.58 86.36 0)
       (effects (font (size 1.27 1.27)) hide)
     )
@@
       (effects (font (size 1.27 1.27)) (justify left))
     )
-    (property "Footprint" "" (id 2) (at 240.03 88.9 0)
+    (property "Footprint" "PrjLibrary:DIP-16_W7.62mm_D1mm" (id 2) (at 240.03 88.9 0)
       (effects (font (size 1.27 1.27)) hide)
     )
@@
       (effects (font (size 1.27 1.27)) (justify left))
     )
-    (property "Footprint" "" (id 2) (at 191.4652 148.59 0)
-      (effects (font (size 1.27 1.27)) hide)
-    )
+    (property "Footprint" "Capacitor_SMD:C_0805_2012Metric_Pad1.18x1.45mm_HandSolder" (id 2) (at 191.4652 148.59 0)
+      (effects (font (size 1.27 1.27)) hide)
+    )
