File: calico_cpu/port_interface.kicad_sch (KiCad schematic)
At the start: 30 parts, among them J3 Conn_02x06_Top_Bottom, J4 Conn_02x06_Top_Bottom, U58 74HC126, U59 74HC126, U60 74HC126, U61 74HC126, U62 74HC273, U63 74HC273

Commit message: calico_cpu: assign footprints
Parts:
- C58, C59, C60, C61, C62, C63: footprint (none) -> Capacitor_SMD:C_0805_2012Metric_Pad1.18x1.45mm_HandSolder
- J3, J4: footprint (none) -> PrjLibrary:PinHeader_2x06_P2.54mm_Vertical_Top_Bottom
- R49, R50, R51, R52, R53, R54, R55, R56, R57, R58, R59, R60, R61, R62, R63, R64: footprint (none) -> Resistor_SMD:R_0805_2012Metric_Pad1.20x1.40mm_HandSolder
- U58, U59, U60, U61: footprint (none) -> PrjLibrary:DIP-14_W7.62mm_D1mm
- U62, U63: footprint (none) -> PrjLibrary:DIP-20_W7.62mm_D1mm
