File: boards/calico_cpu/logic_mux.kicad_sch (KiCad schematic)
At the start: 12 parts, among them U40 74HC153, U41 74HC153, U42 74HC153, U43 74HC153, U44 74HC157, U45 74HC157

Commit message: unify libraries
Parts:
- U40, U41, U42, U43, U44, U45: footprint PrjLibrary:DIP-16_W7.62mm_D1mm -> ModifiedKiCadLibrary:DIP-16_W7.62mm_D1mm
Changed lines of the file:
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@@
       (effects (font (size 1.27 1.27)) (justify left))
     )
-    (property "Footprint" "PrjLibrary:DIP-16_W7.62mm_D1mm" (id 2) (at 185.42 49.53 0)
+    (property "Footprint" "ModifiedKiCadLibrary:DIP-16_W7.62mm_D1mm" (id 2) (at 185.42 49.53 0)
       (effects (font (size 1.27 1.27)) hide)
     )
@@
       (effects (font (size 1.27 1.27)) (justify left))
     )
-    (property "Footprint" "PrjLibrary:DIP-16_W7.62mm_D1mm" (id 2) (at 185.42 121.92 0)
+    (property "Footprint" "ModifiedKiCadLibrary:DIP-16_W7.62mm_D1mm" (id 2) (at 185.42 121.92 0)
       (effects (font (size 1.27 1.27)) hide)
     )
@@
       (effects (font (size 1.27 1.27)) (justify left))
     )
-    (property "Footprint" "PrjLibrary:DIP-16_W7.62mm_D1mm" (id 2) (at 241.3 49.53 0)
+    (property "Footprint" "ModifiedKiCadLibrary:DIP-16_W7.62mm_D1mm" (id 2) (at 241.3 49.53 0)
       (effects (font (size 1.27 1.27)) hide)
     )
@@
       (effects (font (size 1.27 1.27)) (justify left))
     )
-    (property "Footprint" "PrjLibrary:DIP-16_W7.62mm_D1mm" (id 2) (at 241.3 121.92 0)
+    (property "Footprint" "ModifiedKiCadLibrary:DIP-16_W7.62mm_D1mm" (id 2) (at 241.3 121.92 0)
       (effects (font (size 1.27 1.27)) hide)
     )
@@
       (effects (font (size 1.27 1.27)) (justify left))
     )
-    (property "Footprint" "PrjLibrary:DIP-16_W7.62mm_D1mm" (id 2) (at 124.46 49.53 0)
+    (property "Footprint" "ModifiedKiCadLibrary:DIP-16_W7.62mm_D1mm" (id 2) (at 124.46 49.53 0)
       (effects (font (size 1.27 1.27)) hide)
     )
@@
       (effects (font (size 1.27 1.27)) (justify left))
     )
-    (property "Footprint" "PrjLibrary:DIP-16_W7.62mm_D1mm" (id 2) (at 68.58 49.53 0)
-      (effects (font (size 1.27 1.27)) hide)
-    )
+    (property "Footprint" "ModifiedKiCadLibrary:DIP-16_W7.62mm_D1mm" (id 2) (at 68.58 49.53 0)
+      (effects (font (size 1.27 1.27)) hide)
+    )
