File: boards/calico_cpu/logic_rr00ss0x.kicad_sch (KiCad schematic)
At the start: 8 parts, among them U20 74HC08, U21 74HC08, U22 74HC283, U23 74HC283

Commit message: unify libraries
Parts:
- U20, U21: footprint PrjLibrary:DIP-14_W7.62mm_D1mm -> ModifiedKiCadLibrary:DIP-14_W7.62mm_D1mm
- U22, U23: footprint PrjLibrary:DIP-16_W7.62mm_D1mm -> ModifiedKiCadLibrary:DIP-16_W7.62mm_D1mm
Changed lines of the file:
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@@
       (effects (font (size 1.27 1.27)) (justify left))
     )
-    (property "Footprint" "PrjLibrary:DIP-16_W7.62mm_D1mm" (id 2) (at 241.3 95.25 0)
+    (property "Footprint" "ModifiedKiCadLibrary:DIP-16_W7.62mm_D1mm" (id 2) (at 241.3 95.25 0)
       (effects (font (size 1.27 1.27)) hide)
     )
@@
     (property "Reference" "U21" (id 0) (at 115.57 99.06 0))
     (property "Value" "74HC08" (id 1) (at 115.57 101.6 0))
-    (property "Footprint" "PrjLibrary:DIP-14_W7.62mm_D1mm" (id 2) (at 115.57 107.95 0)
+    (property "Footprint" "ModifiedKiCadLibrary:DIP-14_W7.62mm_D1mm" (id 2) (at 115.57 107.95 0)
       (effects (font (size 1.27 1.27)) hide)
     )
@@
     (property "Reference" "U20" (id 0) (at 71.12 114.3 0))
     (property "Value" "74HC08" (id 1) (at 71.12 116.84 0))
-    (property "Footprint" "PrjLibrary:DIP-14_W7.62mm_D1mm" (id 2) (at 71.12 123.19 0)
+    (property "Footprint" "ModifiedKiCadLibrary:DIP-14_W7.62mm_D1mm" (id 2) (at 71.12 123.19 0)
       (effects (font (size 1.27 1.27)) hide)
     )
@@
       (effects (font (size 1.27 1.27)) (justify left))
     )
-    (property "Footprint" "PrjLibrary:DIP-14_W7.62mm_D1mm" (id 2) (at 29.21 173.99 0)
+    (property "Footprint" "ModifiedKiCadLibrary:DIP-14_W7.62mm_D1mm" (id 2) (at 29.21 173.99 0)
       (effects (font (size 1.27 1.27)) hide)
     )
@@
     (property "Reference" "U21" (id 0) (at 115.57 114.3 0))
     (property "Value" "74HC08" (id 1) (at 115.57 116.84 0))
-    (property "Footprint" "PrjLibrary:DIP-14_W7.62mm_D1mm" (id 2) (at 115.57 123.19 0)
+    (property "Footprint" "ModifiedKiCadLibrary:DIP-14_W7.62mm_D1mm" (id 2) (at 115.57 123.19 0)
       (effects (font (size 1.27 1.27)) hide)
     )
@@
     (property "Reference" "U20" (id 0) (at 71.12 68.58 0))
     (property "Value" "74HC08" (id 1) (at 71.12 71.12 0))
-    (property "Footprint" "PrjLibrary:DIP-14_W7.62mm_D1mm" (id 2) (at 71.12 77.47 0)
+    (property "Footprint" "ModifiedKiCadLibrary:DIP-14_W7.62mm_D1mm" (id 2) (at 71.12 77.47 0)
       (effects (font (size 1.27 1.27)) hide)
     )
@@
     (property "Reference" "U20" (id 0) (at 71.12 83.82 0))
     (property "Value" "74HC08" (id 1) (at 71.12 86.36 0))
-    (property "Footprint" "PrjLibrary:DIP-14_W7.62mm_D1mm" (id 2) (at 71.12 92.71 0)
+    (property "Footprint" "ModifiedKiCadLibrary:DIP-14_W7.62mm_D1mm" (id 2) (at 71.12 92.71 0)
       (effects (font (size 1.27 1.27)) hide)
     )
@@
     (property "Reference" "U20" (id 0) (at 71.12 99.06 0))
     (property "Value" "74HC08" (id 1) (at 71.12 101.6 0))
-    (property "Footprint" "PrjLibrary:DIP-14_W7.62mm_D1mm" (id 2) (at 71.12 107.95 0)
+    (property "Footprint" "ModifiedKiCadLibrary:DIP-14_W7.62mm_D1mm" (id 2) (at 71.12 107.95 0)
       (effects (font (size 1.27 1.27)) hide)
     )
@@
     (property "Reference" "U21" (id 0) (at 115.57 68.58 0))
     (property "Value" "74HC08" (id 1) (at 115.57 71.12 0))
-    (property "Footprint" "PrjLibrary:DIP-14_W7.62mm_D1mm" (id 2) (at 115.57 77.47 0)
+    (property "Footprint" "ModifiedKiCadLibrary:DIP-14_W7.62mm_D1mm" (id 2) (at 115.57 77.47 0)
       (effects (font (size 1.27 1.27)) hide)
     )
@@
       (effects (font (size 1.27 1.27)) (justify left))
     )
-    (property "Footprint" "PrjLibrary:DIP-16_W7.62mm_D1mm" (id 2) (at 185.42 95.25 0)
+    (property "Footprint" "ModifiedKiCadLibrary:DIP-16_W7.62mm_D1mm" (id 2) (at 185.42 95.25 0)
       (effects (font (size 1.27 1.27)) hide)
     )
@@
       (effects (font (size 1.27 1.27)) (justify left))
     )
-    (property "Footprint" "PrjLibrary:DIP-14_W7.62mm_D1mm" (id 2) (at 53.34 173.99 0)
+    (property "Footprint" "ModifiedKiCadLibrary:DIP-14_W7.62mm_D1mm" (id 2) (at 53.34 173.99 0)
       (effects (font (size 1.27 1.27)) hide)
     )
@@
     (property "Reference" "U21" (id 0) (at 115.57 83.82 0))
     (property "Value" "74HC08" (id 1) (at 115.57 86.36 0))
-    (property "Footprint" "PrjLibrary:DIP-14_W7.62mm_D1mm" (id 2) (at 115.57 92.71 0)
-      (effects (font (size 1.27 1.27)) hide)
-    )
+    (property "Footprint" "ModifiedKiCadLibrary:DIP-14_W7.62mm_D1mm" (id 2) (at 115.57 92.71 0)
+      (effects (font (size 1.27 1.27)) hide)
+    )
