File: boards/calico_cpu/logic_rr1xvvvv.kicad_sch (KiCad schematic)
At the start: 8 parts, among them U36 74HC08, U37 74HC283, U38 74HC283, U39 74HC08

Commit message: unify libraries
Parts:
- U36, U39: footprint PrjLibrary:DIP-14_W7.62mm_D1mm -> ModifiedKiCadLibrary:DIP-14_W7.62mm_D1mm
- U37, U38: footprint PrjLibrary:DIP-16_W7.62mm_D1mm -> ModifiedKiCadLibrary:DIP-16_W7.62mm_D1mm
Changed lines of the file:
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@@
     (property "Reference" "U39" (id 0) (at 247.65 90.17 0))
     (property "Value" "74HC08" (id 1) (at 247.65 92.71 0))
-    (property "Footprint" "PrjLibrary:DIP-14_W7.62mm_D1mm" (id 2) (at 247.65 99.06 0)
+    (property "Footprint" "ModifiedKiCadLibrary:DIP-14_W7.62mm_D1mm" (id 2) (at 247.65 99.06 0)
       (effects (font (size 1.27 1.27)) hide)
     )
@@
       (effects (font (size 1.27 1.27)) (justify left))
     )
-    (property "Footprint" "PrjLibrary:DIP-14_W7.62mm_D1mm" (id 2) (at 66.04 165.1 0)
+    (property "Footprint" "ModifiedKiCadLibrary:DIP-14_W7.62mm_D1mm" (id 2) (at 66.04 165.1 0)
       (effects (font (size 1.27 1.27)) hide)
     )
@@
       (effects (font (size 1.27 1.27)) (justify left))
     )
-    (property "Footprint" "PrjLibrary:DIP-16_W7.62mm_D1mm" (id 2) (at 132.08 90.17 0)
+    (property "Footprint" "ModifiedKiCadLibrary:DIP-16_W7.62mm_D1mm" (id 2) (at 132.08 90.17 0)
       (effects (font (size 1.27 1.27)) hide)
     )
@@
     (property "Reference" "U39" (id 0) (at 247.65 74.93 0))
     (property "Value" "74HC08" (id 1) (at 247.65 77.47 0))
-    (property "Footprint" "PrjLibrary:DIP-14_W7.62mm_D1mm" (id 2) (at 247.65 83.82 0)
+    (property "Footprint" "ModifiedKiCadLibrary:DIP-14_W7.62mm_D1mm" (id 2) (at 247.65 83.82 0)
       (effects (font (size 1.27 1.27)) hide)
     )
@@
     (property "Reference" "U36" (id 0) (at 83.82 59.69 0))
     (property "Value" "74HC08" (id 1) (at 83.82 62.23 0))
-    (property "Footprint" "PrjLibrary:DIP-14_W7.62mm_D1mm" (id 2) (at 83.82 68.58 0)
+    (property "Footprint" "ModifiedKiCadLibrary:DIP-14_W7.62mm_D1mm" (id 2) (at 83.82 68.58 0)
       (effects (font (size 1.27 1.27)) hide)
     )
@@
     (property "Reference" "U36" (id 0) (at 83.82 74.93 0))
     (property "Value" "74HC08" (id 1) (at 83.82 77.47 0))
-    (property "Footprint" "PrjLibrary:DIP-14_W7.62mm_D1mm" (id 2) (at 83.82 83.82 0)
+    (property "Footprint" "ModifiedKiCadLibrary:DIP-14_W7.62mm_D1mm" (id 2) (at 83.82 83.82 0)
       (effects (font (size 1.27 1.27)) hide)
     )
@@
     (property "Reference" "U36" (id 0) (at 83.82 90.17 0))
     (property "Value" "74HC08" (id 1) (at 83.82 92.71 0))
-    (property "Footprint" "PrjLibrary:DIP-14_W7.62mm_D1mm" (id 2) (at 83.82 99.06 0)
+    (property "Footprint" "ModifiedKiCadLibrary:DIP-14_W7.62mm_D1mm" (id 2) (at 83.82 99.06 0)
       (effects (font (size 1.27 1.27)) hide)
     )
@@
     (property "Reference" "U36" (id 0) (at 83.82 105.41 0))
     (property "Value" "74HC08" (id 1) (at 83.82 107.95 0))
-    (property "Footprint" "PrjLibrary:DIP-14_W7.62mm_D1mm" (id 2) (at 83.82 114.3 0)
+    (property "Footprint" "ModifiedKiCadLibrary:DIP-14_W7.62mm_D1mm" (id 2) (at 83.82 114.3 0)
       (effects (font (size 1.27 1.27)) hide)
     )
@@
       (effects (font (size 1.27 1.27)) (justify left))
     )
-    (property "Footprint" "PrjLibrary:DIP-14_W7.62mm_D1mm" (id 2) (at 41.91 165.1 0)
+    (property "Footprint" "ModifiedKiCadLibrary:DIP-14_W7.62mm_D1mm" (id 2) (at 41.91 165.1 0)
       (effects (font (size 1.27 1.27)) hide)
     )
@@
       (effects (font (size 1.27 1.27)) (justify left))
     )
-    (property "Footprint" "PrjLibrary:DIP-16_W7.62mm_D1mm" (id 2) (at 187.96 90.17 0)
+    (property "Footprint" "ModifiedKiCadLibrary:DIP-16_W7.62mm_D1mm" (id 2) (at 187.96 90.17 0)
       (effects (font (size 1.27 1.27)) hide)
     )
@@
     (property "Reference" "U39" (id 0) (at 247.65 105.41 0))
     (property "Value" "74HC08" (id 1) (at 247.65 107.95 0))
-    (property "Footprint" "PrjLibrary:DIP-14_W7.62mm_D1mm" (id 2) (at 247.65 114.3 0)
+    (property "Footprint" "ModifiedKiCadLibrary:DIP-14_W7.62mm_D1mm" (id 2) (at 247.65 114.3 0)
       (effects (font (size 1.27 1.27)) hide)
     )
@@
     (property "Reference" "U39" (id 0) (at 247.65 59.69 0))
     (property "Value" "74HC08" (id 1) (at 247.65 62.23 0))
-    (property "Footprint" "PrjLibrary:DIP-14_W7.62mm_D1mm" (id 2) (at 247.65 68.58 0)
-      (effects (font (size 1.27 1.27)) hide)
-    )
+    (property "Footprint" "ModifiedKiCadLibrary:DIP-14_W7.62mm_D1mm" (id 2) (at 247.65 68.58 0)
+      (effects (font (size 1.27 1.27)) hide)
+    )
