File: boards/calico_cpu/regs_mux.kicad_sch (KiCad schematic)
At the start: 16 parts, among them U12 74HC153, U13 74HC153, U14 74HC153, U15 74HC153, U16 74HC153, U17 74HC153, U18 74HC153, U19 74HC153

Commit message: unify libraries
Parts:
- U12, U13, U14, U15, U16, U17, U18, U19: footprint PrjLibrary:DIP-16_W7.62mm_D1mm -> ModifiedKiCadLibrary:DIP-16_W7.62mm_D1mm
Changed lines of the file:
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@@
       (effects (font (size 1.27 1.27)) (justify left))
     )
-    (property "Footprint" "PrjLibrary:DIP-16_W7.62mm_D1mm" (id 2) (at 63.5 123.19 0)
+    (property "Footprint" "ModifiedKiCadLibrary:DIP-16_W7.62mm_D1mm" (id 2) (at 63.5 123.19 0)
       (effects (font (size 1.27 1.27)) hide)
     )
@@
       (effects (font (size 1.27 1.27)) (justify left))
     )
-    (property "Footprint" "PrjLibrary:DIP-16_W7.62mm_D1mm" (id 2) (at 236.22 52.07 0)
+    (property "Footprint" "ModifiedKiCadLibrary:DIP-16_W7.62mm_D1mm" (id 2) (at 236.22 52.07 0)
       (effects (font (size 1.27 1.27)) hide)
     )
@@
       (effects (font (size 1.27 1.27)) (justify left))
     )
-    (property "Footprint" "PrjLibrary:DIP-16_W7.62mm_D1mm" (id 2) (at 119.38 52.07 0)
+    (property "Footprint" "ModifiedKiCadLibrary:DIP-16_W7.62mm_D1mm" (id 2) (at 119.38 52.07 0)
       (effects (font (size 1.27 1.27)) hide)
     )
@@
       (effects (font (size 1.27 1.27)) (justify left))
     )
-    (property "Footprint" "PrjLibrary:DIP-16_W7.62mm_D1mm" (id 2) (at 236.22 123.19 0)
+    (property "Footprint" "ModifiedKiCadLibrary:DIP-16_W7.62mm_D1mm" (id 2) (at 236.22 123.19 0)
       (effects (font (size 1.27 1.27)) hide)
     )
@@
       (effects (font (size 1.27 1.27)) (justify left))
     )
-    (property "Footprint" "PrjLibrary:DIP-16_W7.62mm_D1mm" (id 2) (at 180.34 123.19 0)
+    (property "Footprint" "ModifiedKiCadLibrary:DIP-16_W7.62mm_D1mm" (id 2) (at 180.34 123.19 0)
       (effects (font (size 1.27 1.27)) hide)
     )
@@
       (effects (font (size 1.27 1.27)) (justify left))
     )
-    (property "Footprint" "PrjLibrary:DIP-16_W7.62mm_D1mm" (id 2) (at 119.38 123.19 0)
+    (property "Footprint" "ModifiedKiCadLibrary:DIP-16_W7.62mm_D1mm" (id 2) (at 119.38 123.19 0)
       (effects (font (size 1.27 1.27)) hide)
     )
@@
       (effects (font (size 1.27 1.27)) (justify left))
     )
-    (property "Footprint" "PrjLibrary:DIP-16_W7.62mm_D1mm" (id 2) (at 63.5 52.07 0)
+    (property "Footprint" "ModifiedKiCadLibrary:DIP-16_W7.62mm_D1mm" (id 2) (at 63.5 52.07 0)
       (effects (font (size 1.27 1.27)) hide)
     )
@@
       (effects (font (size 1.27 1.27)) (justify left))
     )
-    (property "Footprint" "PrjLibrary:DIP-16_W7.62mm_D1mm" (id 2) (at 180.34 52.07 0)
-      (effects (font (size 1.27 1.27)) hide)
-    )
+    (property "Footprint" "ModifiedKiCadLibrary:DIP-16_W7.62mm_D1mm" (id 2) (at 180.34 52.07 0)
+      (effects (font (size 1.27 1.27)) hide)
+    )
