File: boards/clock_reset/clock_reset.kicad_pcb (KiCad board)
At the start: 2 copper layers, 85.1 x 64.8 mm, 37 parts, among them J1 USB-MicroB-power, J2 signal_out, J3 uart_conn, J4 ICSP, SW1 green, SW2 yellow, SW3 red, SW4 white, SW5 white, U1 ATmega328P-P, U2 AQM0802A, Y1 16MHz

Commit message: clock_reset: add title
Other:
- board text added: "Clock & Reset Board v1.0"
Changed lines of the file:
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@@
   (gr_line (start 205.74 133.35) (end 120.65 133.35) (layer "Edge.Cuts") (width 0.1))
   (gr_line (start 120.65 68.58) (end 120.65 133.35) (layer "Edge.Cuts") (width 0.1))
+  (gr_text "Clock & Reset Board\nv1.0" (at 203.2 128.27) (layer "B.SilkS")
+    (effects (font (size 1.5 1.5) (thickness 0.2)) (justify left mirror))
+  )
   (gr_text "CLOCK" (at 195.58 80.01) (layer "F.SilkS")
     (effects (font (size 1.7 1.7) (thickness 0.25)))

Commit message: change values according to actual parts
Parts:
- R6: value 5k -> 3.9k
Changed lines of the file:
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@@
       (effects (font (size 1 1) (thickness 0.15)) (justify mirror))
     )
-    (fp_text value "5k" (at 0 -1.65) (layer "B.Fab")
+    (fp_text value "3.9k" (at 0 -1.65) (layer "B.Fab")
       (effects (font (size 1 1) (thickness 0.15)) (justify mirror))
     )

Commit message: unify libraries
Parts:
- J1: footprint PrjLibrary:USB-MicroB-power -> MyLibrary:USB-MicroB-power
- U1: footprint PrjLibrary:DIP-28_W7.62mm-D1mm -> ModifiedKiCadLibrary:DIP-28_W7.62mm-D1mm
- U2: footprint PrjLibrary:AQM0802A-RN-GBW -> MyLibrary:AQM0802A-RN-GBW
Changed lines of the file:
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@@
     )
   )
-  (footprint "PrjLibrary:AQM0802A-RN-GBW" (layer "F.Cu")
+  (footprint "MyLibrary:AQM0802A-RN-GBW" (layer "F.Cu")
     (at 169.26 113.62)
     (property "Sheetfile" "clock_reset.kicad_sch")
@@
       (effects (font (size 1 1) (thickness 0.15)))
     )
-    (fp_text user "${REFERENCE}" (at 6 3.25 unlocked) (layer "F.Fab")
+    (fp_text user "${REFERENCE}" (at 6 -20.275 unlocked) (layer "F.Fab")
       (effects (font (size 1 1) (thickness 0.15)))
     )
-    (fp_line (start -9 -19.5) (end 21 -19.5) (layer "F.SilkS") (width 0.12))
-    (fp_line (start -7.5 -7.5) (end 19.5 -7.5) (layer "F.SilkS") (width 0.12))
-    (fp_line (start -9 0) (end -1 0) (layer "F.SilkS") (width 0.12))
     (fp_line (start 21 -19.5) (end 21 0) (layer "F.SilkS") (width 0.12))
-    (fp_line (start 19.5 -7.5) (end 19.5 -18) (layer "F.SilkS") (width 0.12))
-    (fp_line (start 19.5 -18) (end -7.5 -18) (layer "F.SilkS") (width 0.12))
     (fp_line (start -9 0) (end -9 -19.5) (layer "F.SilkS") (width 0.12))
     (fp_line (start 13 0) (end 21 0) (layer "F.SilkS") (width 0.12))
+    (fp_line (start 19.5 -18) (end -7.5 -18) (layer "F.SilkS") (width 0.12))
+    (fp_line (start 19.5 -7.5) (end 19.5 -18) (layer "F.SilkS") (width 0.12))
     (fp_line (start -7.5 -18) (end -7.5 -7.5) (layer "F.SilkS") (width 0.12))
+    (fp_line (start -9 -19.5) (end 21 -19.5) (layer "F.SilkS") (width 0.12))
+    (fp_line (start -9 0) (end -1 0) (layer "F.SilkS") (width 0.12))
+    (fp_line (start -7.5 -7.5) (end 19.5 -7.5) (layer "F.SilkS") (width 0.12))
     (pad "1" thru_hole oval (at 0 0) (size 1.15 2) (drill 0.8 (offset 0 -0.4)) (layers *.Cu *.Mask)
       (net 30 "unconnected-(U2-Pad1)") (pinfunction "VO") (pintype "passive+no_connect"))
@@
     )
   )
-  (footprint "PrjLibrary:USB-MicroB-power" (layer "F.Cu")
+  (footprint "MyLibrary:USB-MicroB-power" (layer "F.Cu")
     (at 123.825 126.365 -90)
     (property "Sheetfile" "clock_reset.kicad_sch")
@@
     )
     (fp_line (start 3.5 1.5) (end 3.5 2.5) (layer "F.SilkS") (width 0.12))
+    (fp_line (start 3.5 -4) (end 2.5 -4) (layer "F.SilkS") (width 0.12))
+    (fp_line (start -3.5 -4) (end -2.5 -4) (layer "F.SilkS") (width 0.12))
+    (fp_line (start 3.5 -1.5) (end 3.5 -4) (layer "F.SilkS") (width 0.12))
+    (fp_line (start -3.5 -1.5) (end -3.5 -4) (layer "F.SilkS") (width 0.12))
     (fp_line (start -3.5 1.5) (end -3.5 2.5) (layer "F.SilkS") (width 0.12))
-    (fp_line (start 3.5 -1.5) (end 3.5 -4) (layer "F.SilkS") (width 0.12))
-    (fp_line (start 3.5 -4) (end 2.5 -4) (layer "F.SilkS") (width 0.12))
-    (fp_line (start -3.5 -1.5) (end -3.5 -4) (layer "F.SilkS") (width 0.12))
-    (fp_line (start -3.5 -4) (end -2.5 -4) (layer "F.SilkS") (width 0.12))
     (fp_line (start 3.5 4) (end 3.5 3) (layer "F.Fab") (width 0.1))
+    (fp_line (start -3.5 3) (end -3.5 4) (layer "F.Fab") (width 0.1))
     (fp_line (start -3.5 4) (end 3.5 4) (layer "F.Fab") (width 0.1))
-    (fp_line (start -3.5 3) (end -3.5 4) (layer "F.Fab") (width 0.1))
     (pad "1" smd rect (at -1.3 -5.9 270) (size 0.9 4.5) (layers "F.Cu" "F.Paste" "F.Mask")
       (net 2 "VCC") (pinfunction "VBUS") (pintype "passive"))
     (pad "5" smd rect (at 1.3 -5.9 270) (size 0.9 4.5) (layers "F.Cu" "F.Paste" "F.Mask")
       (net 1 "GND") (pinfunction "GND") (pintype "passive"))
+    (pad "6" thru_hole oval (at 3.55 0 270) (size 1.6 2.1) (drill oval 0.6 1.1) (layers *.Cu *.Mask)
+      (net 1 "GND") (pinfunction "SHIELD") (pintype "passive"))
     (pad "6" thru_hole oval (at -3.55 0 270) (size 1.6 2.1) (drill oval 0.6 1.1) (layers *.Cu *.Mask)
-      (net 1 "GND") (pinfunction "SHIELD") (pintype "passive"))
-    (pad "6" thru_hole oval (at 3.55 0 270) (size 1.6 2.1) (drill oval 0.6 1.1) (layers *.Cu *.Mask)
       (net 1 "GND") (pinfunction "SHIELD") (pintype "passive"))
   )
@@
       ) (layer "F.SilkS") (width 0.12) (fill solid))
   )
-  (footprint "PrjLibrary:DIP-28_W7.62mm-D1mm" (layer "F.Cu")
+  (footprint "ModifiedKiCadLibrary:DIP-28_W7.62mm-D1mm" (layer "F.Cu")
     (at 152.4 82.55 90)
     (descr "28-lead though-hole mounted DIP package, row spacing 7.62 mm (300 mils) (modified from KiCad 6 library)")
@@
     )
     (fp_line (start 1.16 34.35) (end 6.46 34.35) (layer "F.SilkS") (width 0.12))
+    (fp_line (start 6.46 34.35) (end 6.46 -1.33) (layer "F.SilkS") (width 0.12))
     (fp_line (start 6.46 -1.33) (end 4.81 -1.33) (layer "F.SilkS") (width 0.12))
+    (fp_line (start 1.16 -1.33) (end 1.16 34.35) (layer "F.SilkS") (width 0.12))
     (fp_line (start 2.81 -1.33) (end 1.16 -1.33) (layer "F.SilkS") (width 0.12))
-    (fp_line (start 6.46 34.35) (end 6.46 -1.33) (layer "F.SilkS") (width 0.12))
-    (fp_line (start 1.16 -1.33) (end 1.16 34.35) (layer "F.SilkS") (width 0.12))
     (fp_arc (start 4.81 -1.33) (mid 3.81 -0.33) (end 2.81 -1.33) (layer "F.SilkS") (width 0.12))
+    (fp_line (start 8.7 -1.55) (end -1.1 -1.55) (layer "F.CrtYd") (width 0.05))
+    (fp_line (start -1.1 -1.55) (end -1.1 34.55) (layer "F.CrtYd") (width 0.05))
+    (fp_line (start 8.7 34.55) (end 8.7 -1.55) (layer "F.CrtYd") (width 0.05))
     (fp_line (start -1.1 34.55) (end 8.7 34.55) (layer "F.CrtYd") (width 0.05))
-    (fp_line (start -1.1 -1.55) (end -1.1 34.55) (layer "F.CrtYd") (width 0.05))
-    (fp_line (start 8.7 -1.55) (end -1.1 -1.55) (layer "F.CrtYd") (width 0.05))
-    (fp_line (start 8.7 34.55) (end 8.7 -1.55) (layer "F.CrtYd") (width 0.05))
+    (fp_line (start 1.635 -1.27) (end 6.985 -1.27) (layer "F.Fab") (width 0.1))
+    (fp_line (start 0.635 -0.27) (end 1.635 -1.27) (layer "F.Fab") (width 0.1))
     (fp_line (start 6.985 34.29) (end 0.635 34.29) (layer "F.Fab") (width 0.1))
     (fp_line (start 6.985 -1.27) (end 6.985 34.29) (layer "F.Fab") (width 0.1))
-    (fp_line (start 1.635 -1.27) (end 6.985 -1.27) (layer "F.Fab") (width 0.1))
-    (fp_line (start 0.635 -0.27) (end 1.635 -1.27) (layer "F.Fab") (width 0.1))
     (fp_line (start 0.635 34.29) (end 0.635 -0.27) (layer "F.Fab") (width 0.1))
     (pad "1" thru_hole rect (at 0 0 90) (size 1.7 1.7) (drill 1) (layers *.Cu *.Mask)
