File: boards/kageki/kageki.kicad_pcb (KiCad board)
At the start: 2 copper layers, 99.1 x 99.1 mm, 83 parts, among them J1 Conn_01x06, J2 Conn_02x10_Top_Bottom, J3 Conn_01x06, J4 Conn_01x06, SW1 SW_DIP_x04, U1 74HC161, U10 74HC283, U2 74HC161, U3 74HC161, U4 74HC161, U5 74HC74, U6 74HC138, U7 74HC00, U8 74HC153, U9 74HC153

Commit message: change values according to actual parts
Parts:
- R1, R10, R11, R12, R2, R3, R4, R5, R6, R7, R8, R9: value 20k -> 22k
- R13, R14, R15, R16, R17, R18, R19, R20: value 5k -> 3.9k
Changed lines of the file:
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@@
       (effects (font (size 1 1) (thickness 0.15)) (justify mirror))
     )
-    (fp_text value "20k" (at 0 -1.65 90) (layer "B.Fab")
+    (fp_text value "22k" (at 0 -1.65 90) (layer "B.Fab")
       (effects (font (size 1 1) (thickness 0.15)) (justify mirror))
     )
@@
       (effects (font (size 1 1) (thickness 0.15)) (justify mirror))
     )
-    (fp_text value "20k" (at 0 -1.65) (layer "B.Fab")
+    (fp_text value "22k" (at 0 -1.65) (layer "B.Fab")
       (effects (font (size 1 1) (thickness 0.15)) (justify mirror))
     )
@@
       (effects (font (size 1 1) (thickness 0.15)) (justify mirror))
     )
-    (fp_text value "5k" (at 0 -1.65) (layer "B.Fab")
+    (fp_text value "3.9k" (at 0 -1.65) (layer "B.Fab")
       (effects (font (size 1 1) (thickness 0.15)) (justify mirror))
     )
@@
       (effects (font (size 1 1) (thickness 0.15)) (justify mirror))
     )
-    (fp_text value "5k" (at 0 -1.65 90) (layer "B.Fab")
+    (fp_text value "3.9k" (at 0 -1.65 90) (layer "B.Fab")
       (effects (font (size 1 1) (thickness 0.15)) (justify mirror))
     )
@@
       (effects (font (size 1 1) (thickness 0.15)) (justify mirror))
     )
-    (fp_text value "20k" (at 0 -1.65) (layer "B.Fab")
+    (fp_text value "22k" (at 0 -1.65) (layer "B.Fab")
       (effects (font (size 1 1) (thickness 0.15)) (justify mirror))
     )
@@
       (effects (font (size 1 1) (thickness 0.15)) (justify mirror))
     )
-    (fp_text value "5k" (at 0 -1.65) (layer "B.Fab")
+    (fp_text value "3.9k" (at 0 -1.65) (layer "B.Fab")
       (effects (font (size 1 1) (thickness 0.15)) (justify mirror))
     )
@@
       (effects (font (size 1 1) (thickness 0.15)) (justify mirror))
     )
-    (fp_text value "20k" (at 0 -1.65 90) (layer "B.Fab")
+    (fp_text value "22k" (at 0 -1.65 90) (layer "B.Fab")
       (effects (font (size 1 1) (thickness 0.15)) (justify mirror))
     )
@@
       (effects (font (size 1 1) (thickness 0.15)) (justify mirror))
     )
-    (fp_text value "20k" (at 0 -1.65 90) (layer "B.Fab")
+    (fp_text value "22k" (at 0 -1.65 90) (layer "B.Fab")
       (effects (font (size 1 1) (thickness 0.15)) (justify mirror))
     )
@@
       (effects (font (size 1 1) (thickness 0.15)) (justify mirror))
     )
-    (fp_text value "20k" (at 0 -1.65 90) (layer "B.Fab")
+    (fp_text value "22k" (at 0 -1.65 90) (layer "B.Fab")
       (effects (font (size 1 1) (thickness 0.15)) (justify mirror))
     )
@@
       (effects (font (size 1 1) (thickness 0.15)) (justify mirror))
     )
-    (fp_text value "5k" (at 0 -1.65 90) (layer "B.Fab")
+    (fp_text value "3.9k" (at 0 -1.65 90) (layer "B.Fab")
       (effects (font (size 1 1) (thickness 0.15)) (justify mirror))
     )
@@
       (effects (font (size 1 1) (thickness 0.15)) (justify mirror))
     )
-    (fp_text value "5k" (at 0 -1.65 90) (layer "B.Fab")
+    (fp_text value "3.9k" (at 0 -1.65 90) (layer "B.Fab")
       (effects (font (size 1 1) (thickness 0.15)) (justify mirror))
     )
@@
       (effects (font (size 1 1) (thickness 0.15)) (justify mirror))
     )
-    (fp_text value "20k" (at 0 -1.65 90) (layer "B.Fab")
+    (fp_text value "22k" (at 0 -1.65 90) (layer "B.Fab")
       (effects (font (size 1 1) (thickness 0.15)) (justify mirror))
     )
@@
       (effects (font (size 1 1) (thickness 0.15)) (justify mirror))
     )
-    (fp_text value "5k" (at 0 -1.65 90) (layer "B.Fab")
+    (fp_text value "3.9k" (at 0 -1.65 90) (layer "B.Fab")
       (effects (font (size 1 1) (thickness 0.15)) (justify mirror))
     )
@@
       (effects (font (size 1 1) (thickness 0.15)) (justify mirror))
     )
-    (fp_text value "20k" (at 0 -1.65 90) (layer "B.Fab")
+    (fp_text value "22k" (at 0 -1.65 90) (layer "B.Fab")
       (effects (font (size 1 1) (thickness 0.15)) (justify mirror))
     )
@@
       (effects (font (size 1 1) (thickness 0.15)) (justify mirror))
     )
-    (fp_text value "20k" (at 0 -1.65) (layer "B.Fab")
+    (fp_text value "22k" (at 0 -1.65) (layer "B.Fab")
       (effects (font (size 1 1) (thickness 0.15)) (justify mirror))
     )
@@
       (effects (font (size 1 1) (thickness 0.15)) (justify mirror))
     )
-    (fp_text value "20k" (at 0 -1.65 90) (layer "B.Fab")
+    (fp_text value "22k" (at 0 -1.65 90) (layer "B.Fab")
       (effects (font (size 1 1) (thickness 0.15)) (justify mirror))
     )
@@
       (effects (font (size 1 1) (thickness 0.15)) (justify mirror))
     )
-    (fp_text value "20k" (at 0 -1.65) (layer "B.Fab")
+    (fp_text value "22k" (at 0 -1.65) (layer "B.Fab")
       (effects (font (size 1 1) (thickness 0.15)) (justify mirror))
     )
@@
       (effects (font (size 1 1) (thickness 0.15)) (justify mirror))
     )
-    (fp_text value "20k" (at 0 -1.65 90) (layer "B.Fab")
+    (fp_text value "22k" (at 0 -1.65 90) (layer "B.Fab")
       (effects (font (size 1 1) (thickness 0.15)) (justify mirror))
     )
@@
       (effects (font (size 1 1) (thickness 0.15)) (justify mirror))
     )
-    (fp_text value "5k" (at 0 -1.65) (layer "B.Fab")
+    (fp_text value "3.9k" (at 0 -1.65) (layer "B.Fab")
       (effects (font (size 1 1) (thickness 0.15)) (justify mirror))
     )
@@
       (effects (font (size 1 1) (thickness 0.15)) (justify mirror))
     )
-    (fp_text value "5k" (at 0 -1.65) (layer "B.Fab")
-      (effects (font (size 1 1) (thickness 0.15)) (justify mirror))
-    )
+    (fp_text value "3.9k" (at 0 -1.65) (layer "B.Fab")
+      (effects (font (size 1 1) (thickness 0.15)) (justify mirror))
+    )

Commit message: unify libraries
Parts:
- J2: footprint PrjLibrary_CalicoCPU:PinHeader_2x10_P2.54mm_Vertical_Top_Bottom -> ModifiedKiCadLibrary:PinHeader_2x10_P2.54mm_Vertical_Top_Bottom
- U1, U10, U2, U3, U4, U6, U8, U9: footprint PrjLibrary_CalicoCPU:DIP-16_W7.62mm_D1mm -> ModifiedKiCadLibrary:DIP-16_W7.62mm_D1mm
- U5, U7: footprint PrjLibrary_CalicoCPU:DIP-14_W7.62mm_D1mm -> ModifiedKiCadLibrary:DIP-14_W7.62mm_D1mm
