File: boards/kageki/regs.kicad_sch (KiCad schematic)
At the start: 14 parts, among them U1 74HC161, U2 74HC161, U3 74HC161, U4 74HC161, U5 74HC74, U6 74HC138, U7 74HC00

Commit message: kageki: add board design
Parts:
- renumbered U4 to U1, U1 to U2, U2 to U3, U3 to U4
Changed lines of the file:
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@@
   (symbol (lib_id "74xx:74LS161") (at 104.14 52.07 0) (unit 1)
     (in_bom yes) (on_board yes) (fields_autoplaced)
-    (property "Reference" "U2" (id 0) (at 106.1594 31.75 0)
+    (property "Reference" "U3" (id 0) (at 106.1594 31.75 0)
       (effects (font (size 1.27 1.27)) (justify left))
     )
@@
   (symbol (lib_id "74xx:74LS161") (at 151.13 52.07 0) (unit 1)
     (in_bom yes) (on_board yes) (fields_autoplaced)
-    (property "Reference" "U3" (id 0) (at 153.1494 31.75 0)
+    (property "Reference" "U4" (id 0) (at 153.1494 31.75 0)
       (effects (font (size 1.27 1.27)) (justify left))
     )
@@
   (symbol (lib_id "74xx:74LS161") (at 57.15 52.07 0) (unit 1)
     (in_bom yes) (on_board yes) (fields_autoplaced)
-    (property "Reference" "U1" (id 0) (at 59.1694 31.75 0)
+    (property "Reference" "U2" (id 0) (at 59.1694 31.75 0)
       (effects (font (size 1.27 1.27)) (justify left))
     )
@@
   (symbol (lib_id "74xx:74LS161") (at 198.12 52.07 0) (unit 1)
     (in_bom yes) (on_board yes) (fields_autoplaced)
-    (property "Reference" "U4" (id 0) (at 200.1394 31.75 0)
+    (property "Reference" "U1" (id 0) (at 200.1394 31.75 0)
       (effects (font (size 1.27 1.27)) (justify left))
     )

Commit message: unify libraries
Parts:
- U1, U2, U3, U4, U6: footprint PrjLibrary_CalicoCPU:DIP-16_W7.62mm_D1mm -> ModifiedKiCadLibrary:DIP-16_W7.62mm_D1mm
- U5, U7: footprint PrjLibrary_CalicoCPU:DIP-14_W7.62mm_D1mm -> ModifiedKiCadLibrary:DIP-14_W7.62mm_D1mm
Changed lines of the file:
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@@
       (effects (font (size 1.27 1.27)) (justify left))
     )
-    (property "Footprint" "PrjLibrary_CalicoCPU:DIP-14_W7.62mm_D1mm" (id 2) (at 57.15 160.02 0)
+    (property "Footprint" "ModifiedKiCadLibrary:DIP-14_W7.62mm_D1mm" (id 2) (at 57.15 160.02 0)
       (effects (font (size 1.27 1.27)) hide)
     )
@@
     (property "Reference" "U7" (id 0) (at 102.87 99.06 0))
     (property "Value" "74HC00" (id 1) (at 102.87 101.6 0))
-    (property "Footprint" "PrjLibrary_CalicoCPU:DIP-14_W7.62mm_D1mm" (id 2) (at 102.87 107.95 0)
+    (property "Footprint" "ModifiedKiCadLibrary:DIP-14_W7.62mm_D1mm" (id 2) (at 102.87 107.95 0)
       (effects (font (size 1.27 1.27)) hide)
     )
@@
       (effects (font (size 1.27 1.27)) (justify left))
     )
-    (property "Footprint" "PrjLibrary_CalicoCPU:DIP-14_W7.62mm_D1mm" (id 2) (at 241.3 67.31 0)
+    (property "Footprint" "ModifiedKiCadLibrary:DIP-14_W7.62mm_D1mm" (id 2) (at 241.3 67.31 0)
       (effects (font (size 1.27 1.27)) hide)
     )
@@
       (effects (font (size 1.27 1.27)) (justify left))
     )
-    (property "Footprint" "PrjLibrary_CalicoCPU:DIP-14_W7.62mm_D1mm" (id 2) (at 260.35 69.85 0)
+    (property "Footprint" "ModifiedKiCadLibrary:DIP-14_W7.62mm_D1mm" (id 2) (at 260.35 69.85 0)
       (effects (font (size 1.27 1.27)) hide)
     )
@@
       (effects (font (size 1.27 1.27)) (justify left))
     )
-    (property "Footprint" "PrjLibrary_CalicoCPU:DIP-16_W7.62mm_D1mm" (id 2) (at 57.15 110.49 0)
+    (property "Footprint" "ModifiedKiCadLibrary:DIP-16_W7.62mm_D1mm" (id 2) (at 57.15 110.49 0)
       (effects (font (size 1.27 1.27)) hide)
     )
@@
       (effects (font (size 1.27 1.27)) (justify left))
     )
-    (property "Footprint" "PrjLibrary_CalicoCPU:DIP-14_W7.62mm_D1mm" (id 2) (at 241.3 41.91 0)
+    (property "Footprint" "ModifiedKiCadLibrary:DIP-14_W7.62mm_D1mm" (id 2) (at 241.3 41.91 0)
       (effects (font (size 1.27 1.27)) hide)
     )
@@
     (property "Reference" "U7" (id 0) (at 102.87 115.57 0))
     (property "Value" "74HC00" (id 1) (at 102.87 118.11 0))
-    (property "Footprint" "PrjLibrary_CalicoCPU:DIP-14_W7.62mm_D1mm" (id 2) (at 102.87 124.46 0)
+    (property "Footprint" "ModifiedKiCadLibrary:DIP-14_W7.62mm_D1mm" (id 2) (at 102.87 124.46 0)
       (effects (font (size 1.27 1.27)) hide)
     )
@@
     (property "Reference" "U7" (id 0) (at 151.13 101.6 0))
     (property "Value" "74HC00" (id 1) (at 151.13 104.14 0))
-    (property "Footprint" "PrjLibrary_CalicoCPU:DIP-14_W7.62mm_D1mm" (id 2) (at 151.13 110.49 0)
+    (property "Footprint" "ModifiedKiCadLibrary:DIP-14_W7.62mm_D1mm" (id 2) (at 151.13 110.49 0)
       (effects (font (size 1.27 1.27)) hide)
     )
@@
       (effects (font (size 1.27 1.27)) (justify left))
     )
-    (property "Footprint" "PrjLibrary_CalicoCPU:DIP-16_W7.62mm_D1mm" (id 2) (at 104.14 52.07 0)
+    (property "Footprint" "ModifiedKiCadLibrary:DIP-16_W7.62mm_D1mm" (id 2) (at 104.14 52.07 0)
       (effects (font (size 1.27 1.27)) hide)
     )
@@
       (effects (font (size 1.27 1.27)) (justify left))
     )
-    (property "Footprint" "PrjLibrary_CalicoCPU:DIP-16_W7.62mm_D1mm" (id 2) (at 151.13 52.07 0)
+    (property "Footprint" "ModifiedKiCadLibrary:DIP-16_W7.62mm_D1mm" (id 2) (at 151.13 52.07 0)
       (effects (font (size 1.27 1.27)) hide)
     )
@@
       (effects (font (size 1.27 1.27)) (justify left))
     )
-    (property "Footprint" "PrjLibrary_CalicoCPU:DIP-16_W7.62mm_D1mm" (id 2) (at 57.15 52.07 0)
+    (property "Footprint" "ModifiedKiCadLibrary:DIP-16_W7.62mm_D1mm" (id 2) (at 57.15 52.07 0)
       (effects (font (size 1.27 1.27)) hide)
     )
@@
       (effects (font (size 1.27 1.27)) (justify left))
     )
-    (property "Footprint" "PrjLibrary_CalicoCPU:DIP-16_W7.62mm_D1mm" (id 2) (at 198.12 52.07 0)
+    (property "Footprint" "ModifiedKiCadLibrary:DIP-16_W7.62mm_D1mm" (id 2) (at 198.12 52.07 0)
       (effects (font (size 1.27 1.27)) hide)
     )
@@
     (property "Reference" "U7" (id 0) (at 127 118.11 0))
     (property "Value" "74HC00" (id 1) (at 127 120.65 0))
-    (property "Footprint" "PrjLibrary_CalicoCPU:DIP-14_W7.62mm_D1mm" (id 2) (at 127 127 0)
-      (effects (font (size 1.27 1.27)) hide)
-    )
+    (property "Footprint" "ModifiedKiCadLibrary:DIP-14_W7.62mm_D1mm" (id 2) (at 127 127 0)
+      (effects (font (size 1.27 1.27)) hide)
+    )
