File: boards/rom_write_shield/rom_write_shield.kicad_sch (KiCad schematic)
At the start: 38 parts, among them J1 Conn_01x08, J2 Conn_01x06, J3 Conn_01x08, J4 Conn_01x06, J5 Conn_02x10_Top_Bottom, J6 Conn_01x02, J7 vraw_test, Q1 2SC1815, U1 LT1930, U2 LM358N

Commit message: unify libraries
Parts:
- J5: footprint PrjLibrary_MainBoard:PinHeader_2x10_P2.54mm_Vertical_Top_Bottom -> ModifiedKiCadLibrary:PinHeader_2x10_P2.54mm_Vertical_Top_Bottom
- RV1, RV2, RV3: footprint PrjLibrary:GF063P -> MyLibrary:GF063P
- U1: symbol PrjLibrary:LT1930 -> MyLibrary:LT1930
- U2: footprint PrjLibrary:DIP-8_W7.62mm_D1mm -> ModifiedKiCadLibrary:DIP-8_W7.62mm_D1mm
Changed lines of the file:
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@@
     (property "Reference" "J5" (id 0) (at 213.36 44.45 0))
     (property "Value" "Conn_02x10_Top_Bottom" (id 1) (at 213.36 46.99 0))
-    (property "Footprint" "PrjLibrary_MainBoard:PinHeader_2x10_P2.54mm_Vertical_Top_Bottom" (id 2) (at 212.09 60.96 0)
+    (property "Footprint" "ModifiedKiCadLibrary:PinHeader_2x10_P2.54mm_Vertical_Top_Bottom" (id 2) (at 212.09 60.96 0)
       (effects (font (size 1.27 1.27)) hide)
     )
@@
       (effects (font (size 1.27 1.27)) (justify right))
     )
-    (property "Footprint" "PrjLibrary:GF063P" (id 2) (at 77.47 86.36 0)
+    (property "Footprint" "MyLibrary:GF063P" (id 2) (at 77.47 86.36 0)
       (effects (font (size 1.27 1.27)) hide)
     )
@@
     (property "Reference" "U2" (id 0) (at 154.94 80.01 0))
     (property "Value" "LM358N" (id 1) (at 154.94 82.55 0))
-    (property "Footprint" "PrjLibrary:DIP-8_W7.62mm_D1mm" (id 2) (at 154.94 90.17 0)
+    (property "Footprint" "ModifiedKiCadLibrary:DIP-8_W7.62mm_D1mm" (id 2) (at 154.94 90.17 0)
       (effects (font (size 1.27 1.27)) hide)
     )
@@
       (effects (font (size 1.27 1.27)) (justify right))
     )
-    (property "Footprint" "PrjLibrary:GF063P" (id 2) (at 137.16 87.63 0)
+    (property "Footprint" "MyLibrary:GF063P" (id 2) (at 137.16 87.63 0)
       (effects (font (size 1.27 1.27)) hide)
     )
@@
     (property "Reference" "RV1" (id 0) (at 104.14 30.48 90))
     (property "Value" "100k" (id 1) (at 104.14 33.02 90))
-    (property "Footprint" "PrjLibrary:GF063P" (id 2) (at 104.14 36.195 0)
+    (property "Footprint" "MyLibrary:GF063P" (id 2) (at 104.14 36.195 0)
       (effects (font (size 1.27 1.27)) hide)
     )
@@
       (effects (font (size 1.27 1.27)) (justify left))
     )
-    (property "Footprint" "PrjLibrary:DIP-8_W7.62mm_D1mm" (id 2) (at 139.7 45.085 0)
+    (property "Footprint" "ModifiedKiCadLibrary:DIP-8_W7.62mm_D1mm" (id 2) (at 139.7 45.085 0)
       (effects (font (size 1.27 1.27)) hide)
     )
@@
     (pin "2")
   )
-  (symbol (lib_id "PrjLibrary:LT1930") (at 83.82 46.355 0) (unit 1)
+  (symbol (lib_id "MyLibrary:LT1930") (at 83.82 46.355 0) (unit 1)
     (in_bom yes) (on_board yes)
     (property "Reference" "U1" (id 0) (at 96.52 43.18 0))
@@
     (property "Reference" "U2" (id 0) (at 106.68 78.74 0))
     (property "Value" "LM358N" (id 1) (at 106.68 81.28 0))
-    (property "Footprint" "PrjLibrary:DIP-8_W7.62mm_D1mm" (id 2) (at 106.68 88.9 0)
+    (property "Footprint" "ModifiedKiCadLibrary:DIP-8_W7.62mm_D1mm" (id 2) (at 106.68 88.9 0)
       (effects (font (size 1.27 1.27)) hide)
     )
@@
     )
     (path "/5bd9bd00-e17c-4137-8daf-974f4e7eb479"
-      (reference "J5") (unit 1) (value "Conn_02x10_Top_Bottom") (footprint "PrjLibrary_MainBoard:PinHeader_2x10_P2.54mm_Vertical_Top_Bottom")
+      (reference "J5") (unit 1) (value "Conn_02x10_Top_Bottom") (footprint "ModifiedKiCadLibrary:PinHeader_2x10_P2.54mm_Vertical_Top_Bottom")
     )
     (path "/8997cf99-8749-44a3-a1ae-a79b697a91cc"
@@
     )
     (path "/81386521-8f9b-411f-9833-1dd6b271ccd8"
-      (reference "RV1") (unit 1) (value "100k") (footprint "PrjLibrary:GF063P")
+      (reference "RV1") (unit 1) (value "100k") (footprint "MyLibrary:GF063P")
     )
     (path "/73a38cf8-037e-4a4f-a07d-0cd8e9bdba5b"
-      (reference "RV2") (unit 1) (value "100k") (footprint "PrjLibrary:GF063P")
+      (reference "RV2") (unit 1) (value "100k") (footprint "MyLibrary:GF063P")
     )
     (path "/65ba9d29-16f5-4195-a8b8-68d5b5a71cca"
-      (reference "RV3") (unit 1) (value "100k") (footprint "PrjLibrary:GF063P")
+      (reference "RV3") (unit 1) (value "100k") (footprint "MyLibrary:GF063P")
     )
     (path "/c4647b4f-988f-4d42-ab8f-2b2fd584d489"
@@
     )
     (path "/728702e3-d0ed-44f7-9d2b-bec1d8a1e355"
-      (reference "U2") (unit 1) (value "LM358N") (footprint "PrjLibrary:DIP-8_W7.62mm_D1mm")
+      (reference "U2") (unit 1) (value "LM358N") (footprint "ModifiedKiCadLibrary:DIP-8_W7.62mm_D1mm")
     )
     (path "/ed31e92a-404a-4406-8b6e-38b515b0aaf8"
-      (reference "U2") (unit 2) (value "LM358N") (footprint "PrjLibrary:DIP-8_W7.62mm_D1mm")
+      (reference "U2") (unit 2) (value "LM358N") (footprint "ModifiedKiCadLibrary:DIP-8_W7.62mm_D1mm")
     )
     (path "/a7d379f7-5ca8-4f08-8489-a94bb142d785"
-      (reference "U2") (unit 3) (value "LM358N") (footprint "PrjLibrary:DIP-8_W7.62mm_D1mm")
-    )
-  )
+      (reference "U2") (unit 3) (value "LM358N") (footprint "ModifiedKiCadLibrary:DIP-8_W7.62mm_D1mm")
+    )
+  )
