File: boards/switch_board/switch_board.kicad_sch (KiCad schematic)
At the start: 10 parts, among them J1 Conn_02x06_Top_Bottom, SW1 SW_DIP_x08

Commit message: unify libraries
Parts:
- J1: footprint PrjLibrary:PinSocket_2x06_P2.54mm_Vertical_Top_Bottom -> ModifiedKiCadLibrary:PinSocket_2x06_P2.54mm_Vertical_Top_Bottom
- SW1: footprint PrjLibrary:SW_DIP_SPSTx08_Slide_9.78x22.5mm_W7.62mm_P2.54mm_short -> ModifiedKiCadLibrary:SW_DIP_SPSTx08_Slide_9.78x22.5mm_W7.62mm_P2.54mm_short
Changed lines of the file:
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@@
     (property "Reference" "J1" (id 0) (at 102.87 69.85 0))
     (property "Value" "Conn_02x06_Top_Bottom" (id 1) (at 102.87 72.39 0))
-    (property "Footprint" "PrjLibrary:PinSocket_2x06_P2.54mm_Vertical_Top_Bottom" (id 2) (at 104.14 81.28 0)
+    (property "Footprint" "ModifiedKiCadLibrary:PinSocket_2x06_P2.54mm_Vertical_Top_Bottom" (id 2) (at 104.14 81.28 0)
       (effects (font (size 1.27 1.27)) hide)
     )
@@
     (property "Reference" "SW1" (id 0) (at 165.1 69.85 0))
     (property "Value" "SW_DIP_x08" (id 1) (at 165.1 72.39 0))
-    (property "Footprint" "PrjLibrary:SW_DIP_SPSTx08_Slide_9.78x22.5mm_W7.62mm_P2.54mm_short" (id 2) (at 165.1 87.63 0)
+    (property "Footprint" "ModifiedKiCadLibrary:SW_DIP_SPSTx08_Slide_9.78x22.5mm_W7.62mm_P2.54mm_short" (id 2) (at 165.1 87.63 0)
       (effects (font (size 1.27 1.27)) hide)
     )
@@
     )
     (path "/41bfbe12-e3f8-4aea-8767-3ff73270eca8"
-      (reference "J1") (unit 1) (value "Conn_02x06_Top_Bottom") (footprint "PrjLibrary:PinSocket_2x06_P2.54mm_Vertical_Top_Bottom")
+      (reference "J1") (unit 1) (value "Conn_02x06_Top_Bottom") (footprint "ModifiedKiCadLibrary:PinSocket_2x06_P2.54mm_Vertical_Top_Bottom")
     )
     (path "/bec20459-b20b-4ddc-a042-24a4102341b9"
@@
     )
     (path "/4f41af0e-af2a-428a-8cd5-08eb643145cb"
-      (reference "SW1") (unit 1) (value "SW_DIP_x08") (footprint "PrjLibrary:SW_DIP_SPSTx08_Slide_9.78x22.5mm_W7.62mm_P2.54mm_short")
-    )
-  )
+      (reference "SW1") (unit 1) (value "SW_DIP_x08") (footprint "ModifiedKiCadLibrary:SW_DIP_SPSTx08_Slide_9.78x22.5mm_W7.62mm_P2.54mm_short")
+    )
+  )
