File: boards/other/eprom_zps/eprom_zps.kicad_pcb (KiCad board)
At the start: 2 copper layers, 86.4 x 36.8 mm, 11 parts, among them J1 Conn_02x10_Top_Bottom, J2 Conn_01x02, U1 27C512, U2 XC6201P502MR-G, U3 74HC74, U4 74HC164

Commit message: release boards
* rom_adapter_for_nucky
* software_rom2
* eprom_zps
* convenient_port_shield
* storage_board
* timer_board
Changed lines of the file:
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@@
     (aux_axis_origin 104.775 90.17)
     (pcbplotparams
-      (layerselection 0x00010fc_ffffffff)
+      (layerselection 0x00010f0_ffffffff)
       (disableapertmacros false)
       (usegerberextensions false)
@@
       (viasonmask false)
       (mode 1)
-      (useauxorigin false)
+      (useauxorigin true)
       (hpglpennumber 1)
       (hpglpenspeed 20)
@@
       (outputformat 1)
       (mirror false)
-      (drillshape 1)
+      (drillshape 0)
       (scaleselection 1)
-      (outputdirectory "")
+      (outputdirectory "../../../../release/20220527-boards-v1.0/_gerver_work/eprom_zps/")
     )
   )
@@
   (net 18 "/adata")
   (net 19 "/aclk")
-  (net 20 "Net-(U1-Pad20)")
-  (net 21 "Net-(U1-Pad22)")
+  (net 20 "Net-(J2-Pad1)")
+  (net 21 "Net-(J2-Pad2)")
   (net 22 "/addr15")
   (net 23 "/addr12")
@@
     (fp_line (start 1 0.625) (end -1 0.625) (layer "F.Fab") (width 0.1))
     (fp_line (start 1 -0.625) (end 1 0.625) (layer "F.Fab") (width 0.1))
-    (pad "1" smd roundrect (at -1.0375 0 270) (size 1.175 1.45) (layers "F.Cu" "F.Paste" "F.Mask") (roundrect_rratio 0.212766)
+    (pad "1" smd roundrect (at -1.0375 0 270) (size 1.175 1.45) (layers "F.Cu" "F.Paste" "F.Mask") (roundrect_rratio 0.2127659574)
       (net 3 "+5V") (pintype "passive"))
-    (pad "2" smd roundrect (at 1.0375 0 270) (size 1.175 1.45) (layers "F.Cu" "F.Paste" "F.Mask") (roundrect_rratio 0.212766)
+    (pad "2" smd roundrect (at 1.0375 0 270) (size 1.175 1.45) (layers "F.Cu" "F.Paste" "F.Mask") (roundrect_rratio 0.2127659574)
       (net 2 "GND") (pintype "passive"))
     (model "${KICAD6_3DMODEL_DIR}/Capacitor_SMD.3dshapes/C_0805_2012Metric.wrl"
@@
       (net 11 "/data7") (pinfunction "D7") (pintype "tri_state"))
     (pad "20" thru_hole oval (at 15.24 20.32 90) (size 2 1.44) (drill 1) (layers *.Cu *.Mask)
-      (net 20 "Net-(U1-Pad20)") (pinfunction "~{CE}") (pintype "input"))
+      (net 20 "Net-(J2-Pad1)") (pinfunction "~{CE}") (pintype "input"))
     (pad "21" thru_hole oval (at 15.24 17.78 90) (size 2 1.44) (drill 1) (layers *.Cu *.Mask)
       (net 26 "/addr10") (pinfunction "A10") (pintype "input"))
     (pad "22" thru_hole oval (at 15.24 15.24 90) (size 2 1.44) (drill 1) (layers *.Cu *.Mask)
-      (net 21 "Net-(U1-Pad22)") (pinfunction "~{OE}") (pintype "input"))
+      (net 21 "Net-(J2-Pad2)") (pinfunction "~{OE}") (pintype "input"))
     (pad "23" thru_hole oval (at 15.24 12.7 90) (size 2 1.44) (drill 1) (layers *.Cu *.Mask)
       (net 27 "/addr11") (pinfunction "A11") (pintype "input"))
@@
     (fp_line (start 1 -0.625) (end 1 0.625) (layer "F.Fab") (width 0.1))
     (fp_line (start -1 -0.625) (end 1 -0.625) (layer "F.Fab") (width 0.1))
-    (pad "1" smd roundrect (at -1.0375 0 270) (size 1.175 1.45) (layers "F.Cu" "F.Paste" "F.Mask") (roundrect_rratio 0.212766)
+    (pad "1" smd roundrect (at -1.0375 0 270) (size 1.175 1.45) (layers "F.Cu" "F.Paste" "F.Mask") (roundrect_rratio 0.2127659574)
       (net 1 "VCC") (pintype "passive"))
-    (pad "2" smd roundrect (at 1.0375 0 270) (size 1.175 1.45) (layers "F.Cu" "F.Paste" "F.Mask") (roundrect_rratio 0.212766)
+    (pad "2" smd roundrect (at 1.0375 0 270) (size 1.175 1.45) (layers "F.Cu" "F.Paste" "F.Mask") (roundrect_rratio 0.2127659574)
       (net 2 "GND") (pintype "passive"))
     (model "${KICAD6_3DMODEL_DIR}/Capacitor_SMD.3dshapes/C_0805_2012Metric.wrl"
@@
     (fp_line (start -0.635 -1.27) (end 1.27 -1.27) (layer "F.Fab") (width 0.1))
     (pad "1" thru_hole rect (at 0 0) (size 1.7 1.7) (drill 1) (layers *.Cu *.Mask)
-      (net 20 "Net-(U1-Pad20)") (pinfunction "Pin_1") (pintype "passive"))
+      (net 20 "Net-(J2-Pad1)") (pinfunction "Pin_1") (pintype "passive"))
     (pad "2" thru_hole oval (at 0 2.54) (size 1.7 1.7) (drill 1) (layers *.Cu *.Mask)
-      (net 21 "Net-(U1-Pad22)") (pinfunction "Pin_2") (pintype "passive"))
+      (net 21 "Net-(J2-Pad2)") (pinfunction "Pin_2") (pintype "passive"))
     (model "${KICAD6_3DMODEL_DIR}/Connector_PinSocket_2.54mm.3dshapes/PinSocket_1x02_P2.54mm_Vertical.wrl"
       (offset (xyz 0 -2.54 -1.7))
@@
     (fp_line (start 1 0.625) (end 1 -0.625) (layer "B.Fab") (width 0.1))
     (fp_line (start -1 -0.625) (end -1 0.625) (layer "B.Fab") (width 0.1))
-    (pad "1" smd roundrect (at -1.0375 0) (size 1.175 1.45) (layers "B.Cu" "B.Paste" "B.Mask") (roundrect_rratio 0.212766)
+    (pad "1" smd roundrect (at -1.0375 0) (size 1.175 1.45) (layers "B.Cu" "B.Paste" "B.Mask") (roundrect_rratio 0.2127659574)
       (net 3 "+5V") (pintype "passive"))
-    (pad "2" smd roundrect (at 1.0375 0) (size 1.175 1.45) (layers "B.Cu" "B.Paste" "B.Mask") (roundrect_rratio 0.212766)
+    (pad "2" smd roundrect (at 1.0375 0) (size 1.175 1.45) (layers "B.Cu" "B.Paste" "B.Mask") (roundrect_rratio 0.2127659574)
       (net 2 "GND") (pintype "passive"))
     (model "${KICAD6_3DMODEL_DIR}/Capacitor_SMD.3dshapes/C_0805_2012Metric.wrl"
@@
     (fp_line (start 1 0.625) (end 1 -0.625) (layer "B.Fab") (width 0.1))
     (fp_line (start 1 -0.625) (end -1 -0.625) (layer "B.Fab") (width 0.1))
-    (pad "1" smd roundrect (at -1.0375 0 180) (size 1.175 1.45) (layers "B.Cu" "B.Paste" "B.Mask") (roundrect_rratio 0.212766)
+    (pad "1" smd roundrect (at -1.0375 0 180) (size 1.175 1.45) (layers "B.Cu" "B.Paste" "B.Mask") (roundrect_rratio 0.2127659574)
       (net 1 "VCC") (pintype "passive"))
-    (pad "2" smd roundrect (at 1.0375 0 180) (size 1.175 1.45) (layers "B.Cu" "B.Paste" "B.Mask") (roundrect_rratio 0.212766)
+    (pad "2" smd roundrect (at 1.0375 0 180) (size 1.175 1.45) (layers "B.Cu" "B.Paste" "B.Mask") (roundrect_rratio 0.2127659574)
       (net 2 "GND") (pintype "passive"))
     (model "${KICAD6_3DMODEL_DIR}/Capacitor_SMD.3dshapes/C_0805_2012Metric.wrl"
@@
     (fp_line (start -1 0.625) (end 1 0.625) (layer "B.Fab") (width 0.1))
     (fp_line (start -1 -0.625) (end -1 0.625) (layer "B.Fab") (width 0.1))
-    (pad "1" smd roundrect (at -1.0375 0) (size 1.175 1.45) (layers "B.Cu" "B.Paste" "B.Mask") (roundrect_rratio 0.212766)
+    (pad "1" smd roundrect (at -1.0375 0) (size 1.175 1.45) (layers "B.Cu" "B.Paste" "B.Mask") (roundrect_rratio 0.2127659574)
       (net 3 "+5V") (pintype "passive"))
-    (pad "2" smd roundrect (at 1.0375 0) (size 1.175 1.45) (layers "B.Cu" "B.Paste" "B.Mask") (roundrect_rratio 0.212766)
+    (pad "2" smd roundrect (at 1.0375 0) (size 1.175 1.45) (layers "B.Cu" "B.Paste" "B.Mask") (roundrect_rratio 0.2127659574)
       (net 2 "GND") (pintype "passive"))
     (model "${KICAD6_3DMODEL_DIR}/Capacitor_SMD.3dshapes/C_0805_2012Metric.wrl"
@@
   (segment (start 113.665 71.755) (end 128.905 71.755) (width 0.3) (layer "B.Cu") (net 22))
   (segment (start 130.81 71.12) (end 142.24 82.55) (width 0.3) (layer "B.Cu") (net 23))
-  (segment (start 142.24 82.55) (end 142.24 82.296) (width 0.3) (layer "B.Cu") (net 23))
   (segment (start 120.65 71.12) (end 130.81 71.12) (width 0.3) (layer "B.Cu") (net 23))
   (segment (start 119.38 69.85) (end 120.65 71.12) (width 0.3) (layer "B.Cu") (net 23))
